Commit message: Cambios en archivos URDF

File: urdf/r6g_steppermotor.urdf (robot description, URDF)
Before this commit: robot r6g_steppermotor, 7 links, 6 joints
Joints:
- joint Joint2: axis 0 0 -1 -> 0 0 1

Commit message: Corrección J3 URDF

File: urdf/r6g_steppermotor.urdf (robot description, URDF)
Before this commit: robot r6g_steppermotor, 7 links, 6 joints
Joints:
- joint Joint3: axis 0 0 -1 -> 0 0 1

Commit message: Ajuste límites por software J5 y J6

File: urdf/r6g_steppermotor.urdf (robot description, URDF)
Before this commit: robot r6g_steppermotor, 7 links, 6 joints
Joints:
- joint Joint5: limit lower=-0.34906585 upper=1.74532925 effort=0 velocity=0 -> lower=-0.1745329 upper=1.57079632 effort=0 velocity=0
- joint Joint6: limit lower=-3.14159265 upper=3.14159265 effort=0 velocity=0 -> lower=-1.570796326 upper=1.570796326 effort=0 velocity=0
